File: main.brd (EAGLE design)
At the start: 160 x 100 mm, 7 parts, among them U1 ESP32-DEVKITC-32D, U3 LSM9DS1

Commit message: nice!
Parts:
- added R1, R10, R11, R12, R2, R5, R6, R7, R8, R9: (no value), rcl:0207/10
- added S1, S10, S11, S12, S2, S5, S6, S7, S8, S9: TL36PO, switch:TL3XPO
- added U$1, U$3, U$4, U$5, U$6: DRV8830, FaBo-Motor:DRV8830
Connections:
- removed net 3V3: U1.1
- new net N$10: R5.1, S5.2
- new net N$11: R6.1, S5.3
- new net N$12: S7.1, S8.2
- new net N$13: R7.1, S7.2
- new net N$14: R8.1, S7.3
- new net N$15: S10.2, S9.1
- new net N$16: R9.1, S9.2
- new net N$17: R10.1, S9.3
- new net N$18: S11.1, S12.2
- new net N$19: R11.1, S11.2
- new net N$20: R12.1, S11.3
- new net N$3: S1.1, S2.2
- new net N$4: R1.1, S1.2
- new net N$5: R2.1, S1.3
- new net N$9: S5.1, S6.2
- new net NO1: U$3.1, U1.29
- new net NO10: U$6.3, U1.8
- new net NO2: U$3.3, U1.30
- new net NO3: U$1.1, U1.31
- new net NO4: U$1.3, U1.32
- new net NO5: U$4.1, U1.33
- new net NO6: U$4.3, U1.34
- new net NO7: U$5.1, U1.5
- new net NO8: U$5.3, U1.6
- new net NO9: U$6.1, U1.7
- new net SCL1: U$5.10, U$6.10
- new net SDA1: U$5.9, U$6.9
- net GND: now also R10.2, R12.2, R2.2, R6.2, R8.2, S10.3, S12.3, S2.3, S6.3, S8.3, U$1.5, U$3.5, U$4.5, U$5.5, U$6.5, U1.1
- net MOTORIN: now also U$1.8, U$3.8, U$4.8, U$5.8, U$6.8
- net MOTOROUT: now also U$1.7, U$3.7, U$4.7, U$5.7, U$6.7
- net SCL: now also U$1.10, U$3.10, U$4.10
- net SDA: now also U$1.9, U$3.9, U$4.9
- net VCC: now also R1.2, R11.2, R5.2, R7.2, R9.2, S10.1, S12.1, S2.1, S6.1, S8.1, U$1.4, U$3.4, U$4.4, U$5.4, U$6.4

Commit message: Good?
Connections:
- new net REG: R3.2, S4.1, U$2.4, U1.1
- net GND: no longer U1.1
- net VCC: no longer R3.2, S4.1, U$2.4
Changed lines of the file:
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@@
 </signal>
 <signal name="VCC">
-<contactref element="U$2" pad="4"/>
-<contactref element="R3" pad="2"/>
-<contactref element="S4" pad="1"/>
 <contactref element="U$1" pad="4"/>
 <contactref element="R1" pad="2"/>
@@
 <wire x1="14.47" y1="-17.48" x2="11.43" y2="-27.94" width="0" layer="19" extent="1-1"/>
 <wire x1="3.81" y1="-17.78" x2="14.47" y2="-17.48" width="0" layer="19" extent="1-1"/>
-<wire x1="41.14" y1="67.61" x2="14.47" y2="-17.48" width="0" layer="19" extent="1-1"/>
-<wire x1="38.1" y1="68.58" x2="41.14" y2="67.61" width="0" layer="19" extent="1-1"/>
-<wire x1="53.34" y1="72.39" x2="41.14" y2="67.61" width="0" layer="19" extent="1-1"/>
 </signal>
 <signal name="MOTOROUT">
@@
 </signal>
 <signal name="GND">
-<contactref element="U1" pad="1"/>
-<contactref element="U3" pad="19"/>
-<contactref element="U3" pad="20"/>
-<contactref element="R4" pad="2"/>
-<contactref element="S4" pad="3"/>
-<contactref element="U$2" pad="5"/>
-<contactref element="U1" pad="20"/>
 <contactref element="R2" pad="2"/>
 <contactref element="S2" pad="3"/>
@@
 <contactref element="S12" pad="3"/>
 <contactref element="U$6" pad="5"/>
+<contactref element="U3" pad="19"/>
+<contactref element="U3" pad="20"/>
+<contactref element="R4" pad="2"/>
+<contactref element="S4" pad="3"/>
+<contactref element="U$2" pad="5"/>
+<contactref element="U1" pad="20"/>
 <wire x1="8.89" y1="-154.94" x2="11.43" y2="-170.18" width="0" layer="19" extent="1-1"/>
 <wire x1="14.97" y1="-154.64" x2="8.89" y2="-154.94" width="0" layer="19" extent="1-1"/>
@@
 <wire x1="8.89" y1="-17.78" x2="11.43" y2="-33.02" width="0" layer="19" extent="1-1"/>
 <wire x1="14.97" y1="-17.48" x2="8.89" y2="-17.78" width="0" layer="19" extent="1-1"/>
-<wire x1="34.29" y1="56.59" x2="14.97" y2="-17.48" width="0" layer="19" extent="1-1"/>
-<wire x1="41.64" y1="67.61" x2="34.29" y2="56.59" width="0" layer="19" extent="1-1"/>
-<wire x1="46.365" y1="71.075" x2="41.64" y2="67.61" width="0" layer="19" extent="1-1"/>
-<wire x1="46.795" y1="71.075" x2="46.365" y2="71.075" width="0" layer="19" extent="1-1"/>
-<wire x1="58.42" y1="72.39" x2="46.795" y2="71.075" width="0" layer="19" extent="1-1"/>
-<wire x1="25.4" y1="68.58" x2="34.29" y2="56.59" width="0" layer="19" extent="1-1"/>
-<wire x1="59.69" y1="56.59" x2="58.42" y2="72.39" width="0" layer="19" extent="1-1"/>
+<wire x1="59.69" y1="56.59" x2="14.97" y2="-17.48" width="0" layer="19" extent="1-1"/>
+<wire x1="58.42" y1="72.39" x2="59.69" y2="56.59" width="0" layer="19" extent="1-1"/>
+<wire x1="46.795" y1="71.075" x2="58.42" y2="72.39" width="0" layer="19" extent="1-1"/>
+<wire x1="46.365" y1="71.075" x2="46.795" y2="71.075" width="0" layer="19" extent="1-1"/>
+<wire x1="41.64" y1="67.61" x2="46.365" y2="71.075" width="0" layer="19" extent="1-1"/>
+<wire x1="25.4" y1="68.58" x2="41.64" y2="67.61" width="0" layer="19" extent="1-1"/>
 </signal>
 <signal name="N$9">
@@
 <wire x1="34.29" y1="43.89" x2="13.97" y2="-120.35" width="0" layer="19" extent="1-1"/>
 </signal>
+<signal name="REG">
+<contactref element="U1" pad="1"/>
+<contactref element="U$2" pad="4"/>
+<contactref element="R3" pad="2"/>
+<contactref element="S4" pad="1"/>
+<wire x1="41.14" y1="67.61" x2="53.34" y2="72.39" width="0" layer="19" extent="1-1"/>
+<wire x1="38.1" y1="68.58" x2="41.14" y2="67.61" width="0" layer="19" extent="1-1"/>
+<wire x1="34.29" y1="56.59" x2="38.1" y2="68.58" width="0" layer="19" extent="1-1"/>
+</signal>
 </signals>

Commit message: dou?
Parts:
- removed R10, R11, R12, R3, R4, R5, R6, R7, R8, R9: (no value), rcl:0207/10
- removed S10, S11, S12, S3, S4, S5, S6, S7, S8, S9: TL36PO, switch:TL3XPO
- removed U$1, U$3, U$4, U$5, U$6: DRV8830, FaBo-Motor:DRV8830
- moved R1 24.1 mm to (6.35, -3.81)
- moved S1 5.08 mm to (6.35, -11.4)
- moved S2 5.08 mm to (6.35, -22.9)
Connections:
- net EXT_5V renamed REGOUT
- removed net N$10: R5.1, S5.2
- removed net N$11: R6.1, S5.3
- removed net N$12: S7.1, S8.2
- removed net N$13: R7.1, S7.2
- removed net N$14: R8.1, S7.3
- removed net N$15: S10.2, S9.1
- removed net N$16: R9.1, S9.2
- removed net N$17: R10.1, S9.3
- removed net N$18: S11.1, S12.2
- removed net N$19: R11.1, S11.2
- removed net N$20: R12.1, S11.3
- removed net N$4: R1.1, S1.2
- removed net N$5: R2.1, S1.3
- removed net N$6: S3.1, S4.2
- removed net N$7: R3.1, S3.2
- removed net N$8: R4.1, S3.3
- removed net N$9: S5.1, S6.2
- removed net REG: R3.2, S4.1, U$2.4, U1.1
- removed net SCL1: U$5.10, U$6.10
- removed net SDA1: U$5.9, U$6.9
- removed net VCC: R1.2, R11.2, R5.2, R7.2, R9.2, S10.1, S12.1, S2.1, S6.1, S8.1, U$1.4, U$3.4, U$4.4, U$5.4, U$6.4
- new net ADC: R1.2, S1.2, S2.2, U1.3
- new net N$21: U1.1, U3.10
- new net REGIN: R1.1, U$2.4
- net GND: now also S1.3; no longer R10.2, R12.2, R4.2, R6.2, R8.2, S10.3, S12.3, S2.3, S4.3, S6.3, S8.3, U$1.5, U$3.5, U$4.5, U$5.5, U$6.5
- net MOTORIN: no longer U$1.8, U$3.8, U$4.8, U$5.8, U$6.8
- net MOTOROUT: no longer U$1.7, U$3.7, U$4.7, U$5.7, U$6.7
- net N$3: now also R2.1, S2.3; no longer S1.1, S2.2
- net NO1: no longer U$3.1
- net NO10: no longer U$6.3
- net NO2: no longer U$3.3
- net NO3: no longer U$1.1
- net NO4: no longer U$1.3
- net NO5: no longer U$4.1
- net NO6: no longer U$4.3
- net NO7: no longer U$5.1
- net NO8: no longer U$5.3
- net NO9: no longer U$6.1
- net SCL: no longer U$1.10, U$3.10, U$4.10
- net SDA: no longer U$1.9, U$3.9, U$4.9
