File: main.sch (EAGLE design)
At the start: 0 parts

Commit message: mmm
Parts:
- added U1: ESP32-DEVKITC-32D, ESP32-DEVKITC-32D:ESP32-DEVKITC-32D
Changed lines of the file:
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@@
 <parts>
 <part name="GND1" library="supply1" library_urn="urn:adsk.eagle:library:371" deviceset="GND" device=""/>
+<part name="GND2" library="supply1" library_urn="urn:adsk.eagle:library:371" deviceset="GND" device=""/>
+<part name="GND3" library="supply1" library_urn="urn:adsk.eagle:library:371" deviceset="GND" device=""/>
+<part name="U1" library="ESP32-DEVKITC-32D" deviceset="ESP32-DEVKITC-32D" device=""/>
 </parts>
 <sheets>
@@
 <attribute name="VALUE" x="33.02" y="33.02" size="1.778" layer="96"/>
 </instance>
+<instance part="GND2" gate="1" x="35.56" y="17.78" smashed="yes">
+<attribute name="VALUE" x="33.02" y="15.24" size="1.778" layer="96"/>
+</instance>
+<instance part="GND3" gate="1" x="35.56" y="0" smashed="yes">
+<attribute name="VALUE" x="33.02" y="-2.54" size="1.778" layer="96"/>
+</instance>
+<instance part="U1" gate="G$1" x="78.74" y="22.86" smashed="yes" rot="MR0">
+<attribute name="NAME" x="93.9972" y="48.9243" size="1.78" layer="95" rot="MR0"/>
+<attribute name="VALUE" x="93.9963" y="-5.1098" size="1.7799" layer="96" rot="MR0"/>
+</instance>
 </instances>

Commit message: madatotyuu
Parts:
- added R3, R4: (no value), rcl:R-EU_0207/10
- added S3, S4: TL36PO, switch:TL36PO
- added U$2: DRV8830, FaBo-Motor:DRV8830
- added U3: LSM9DS1, LSM9DS1_temp:LSM9DS1
Connections:
- new net GND: R4.2, S4.S, U$2.GND, U1.GND3, U3.GND
- new net MOTORIN: U$2.A1
- new net MOTOROUT: U$2.A0
- new net N$1: U$2.OUT2, U1.IO19
- new net N$2: U$2.OUT1, U1.IO18
- new net N$6: S3.O, S4.P
- new net N$7: R3.1, S3.P
- new net N$8: R4.1, S3.S
- new net SCL: U$2.SCL, U1.IO22, U3.SCL/SPC
- new net SDA: U$2.SDA, U1.IO21, U3.SDA/SDI/SDO
- new net VCC: R3.2, S4.O, U$2.VCC

Commit message: nice!
Parts:
- added R1, R10, R11, R12, R2, R5, R6, R7, R8, R9: (no value), rcl:R-EU_0207/10
- added S1, S10, S11, S12, S2, S5, S6, S7, S8, S9: TL36PO, switch:TL36PO
- added U$1, U$3, U$4, U$5, U$6: DRV8830, FaBo-Motor:DRV8830
Connections:
- new net N$10: R5.1, S5.P
- new net N$11: R6.1, S5.S
- new net N$12: S7.O, S8.P
- new net N$13: R7.1, S7.P
- new net N$14: R8.1, S7.S
- new net N$15: S10.P, S9.O
- new net N$16: R9.1, S9.P
- new net N$17: R10.1, S9.S
- new net N$18: S11.O, S12.P
- new net N$19: R11.1, S11.P
- new net N$20: R12.1, S11.S
- new net N$3: S1.O, S2.P
- new net N$4: R1.1, S1.P
- new net N$5: R2.1, S1.S
- new net N$9: S5.O, S6.P
- new net NO1: U$3.OUT2, U1.IO5
- new net NO10: U$6.OUT1, U1.IO33
- new net NO2: U$3.OUT1, U1.IO17
- new net NO3: U$1.OUT2, U1.IO16
- new net NO4: U$1.OUT1, U1.IO4
- new net NO5: U$4.OUT2, U1.IO0
- new net NO6: U$4.OUT1, U1.IO2
- new net NO7: U$5.OUT2, U1.IO34
- new net NO8: U$5.OUT1, U1.IO35
- new net NO9: U$6.OUT2, U1.IO32
- new net SCL1: U$5.SCL, U$6.SCL
- new net SDA1: U$5.SDA, U$6.SDA
- net GND: now also R10.2, R12.2, R2.2, R6.2, R8.2, S10.S, S12.S, S2.S, S6.S, S8.S, U$1.GND, U$3.GND, U$4.GND, U$5.GND, U$6.GND, U1.3V3
- net MOTORIN: now also U$1.A1, U$3.A1, U$4.A1, U$5.A1, U$6.A1
- net MOTOROUT: now also U$1.A0, U$3.A0, U$4.A0, U$5.A0, U$6.A0
- net SCL: now also U$1.SCL, U$3.SCL, U$4.SCL
- net SDA: now also U$1.SDA, U$3.SDA, U$4.SDA
- net VCC: now also R1.2, R11.2, R5.2, R7.2, R9.2, S10.O, S12.O, S2.O, S6.O, S8.O, U$1.VCC, U$3.VCC, U$4.VCC, U$5.VCC, U$6.VCC
Other:
- moved on the sheet: U1

Commit message: Good?
Connections:
- new net REG: R3.2, S4.O, U$2.VCC, U1.3V3
- net GND: no longer U1.3V3
- net VCC: no longer R3.2, S4.O, U$2.VCC

Commit message: dou?
Parts:
- removed R10, R11, R12, R3, R4, R5, R6, R7, R8, R9: (no value), rcl:R-EU_0207/10
- removed S10, S11, S12, S3, S4, S5, S6, S7, S8, S9: TL36PO, switch:TL36PO
- removed U$1, U$3, U$4, U$5, U$6: DRV8830, FaBo-Motor:DRV8830
Connections:
- removed net N$10: R5.1, S5.P
- removed net N$11: R6.1, S5.S
- removed net N$12: S7.O, S8.P
- removed net N$13: R7.1, S7.P
- removed net N$14: R8.1, S7.S
- removed net N$15: S10.P, S9.O
- removed net N$16: R9.1, S9.P
- removed net N$17: R10.1, S9.S
- removed net N$18: S11.O, S12.P
- removed net N$19: R11.1, S11.P
- removed net N$20: R12.1, S11.S
- removed net N$4: R1.1, S1.P
- removed net N$5: R2.1, S1.S
- removed net N$6: S3.O, S4.P
- removed net N$7: R3.1, S3.P
- removed net N$8: R4.1, S3.S
- removed net N$9: S5.O, S6.P
- removed net REG: R3.2, S4.O, U$2.VCC, U1.3V3
- removed net SCL1: U$5.SCL, U$6.SCL
- removed net SDA1: U$5.SDA, U$6.SDA
- removed net VCC: R1.2, R11.2, R5.2, R7.2, R9.2, S10.O, S12.O, S2.O, S6.O, S8.O, U$1.VCC, U$3.VCC, U$4.VCC, U$5.VCC, U$6.VCC
- new net ADC: R1.2, S1.P, S2.P, U1.SENSOR_VP
- new net N$21: U1.3V3, U3.INT_M
- new net REGIN: R1.1, U$2.VCC
- new net REGOUT: U1.EXT_5V
- net GND: now also S1.S; no longer R10.2, R12.2, R4.2, R6.2, R8.2, S10.S, S12.S, S2.S, S4.S, S6.S, S8.S, U$1.GND, U$3.GND, U$4.GND, U$5.GND, U$6.GND
- net MOTORIN: no longer U$1.A1, U$3.A1, U$4.A1, U$5.A1, U$6.A1
- net MOTOROUT: no longer U$1.A0, U$3.A0, U$4.A0, U$5.A0, U$6.A0
- net N$3: now also R2.1, S2.S; no longer S1.O, S2.P
- net NO1: no longer U$3.OUT2
- net NO10: no longer U$6.OUT1
- net NO2: no longer U$3.OUT1
- net NO3: no longer U$1.OUT2
- net NO4: no longer U$1.OUT1
- net NO5: no longer U$4.OUT2
- net NO6: no longer U$4.OUT1
- net NO7: no longer U$5.OUT2
- net NO8: no longer U$5.OUT1
- net NO9: no longer U$6.OUT2
- net SCL: no longer U$1.SCL, U$3.SCL, U$4.SCL
- net SDA: no longer U$1.SDA, U$3.SDA, U$4.SDA
Other:
- moved on the sheet: R1, R2, S1, S2
